File: PCB/ESP.kicad_sch (KiCad schematic)
At the start: 14 parts, among them J4 , SW2 SW_Push, SW3 SW_Push, U10 ESP-07

Commit message: raw placement
Parts:
- J4: footprint Connector_PinHeader_2.54mm:PinHeader_1x06_P2.54mm_Vertical -> IVS_FOOTPRINTS:PinHeader_1x06_P2.54mm_Vertical
Changed lines of the file:
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@@
       (effects (font (size 1.27 1.27)) hide)
     )
-    (property "Footprint" "Connector_PinHeader_2.54mm:PinHeader_1x06_P2.54mm_Vertical" (at 187.96 60.325 0)
+    (property "Footprint" "IVS_FOOTPRINTS:PinHeader_1x06_P2.54mm_Vertical" (at 187.96 60.325 0)
       (effects (font (size 1.27 1.27)) hide)
     )
