File: PCB/Peripheral.kicad_sch (KiCad schematic)
At the start: 89 parts, among them IC1 RTC_DS3231M, J1 Conn_01x03, J11 Conn_01x03_Pin, J13 Conn_01x02_Pin, J2 Conn_01x02, J4 Conn_01x04, J5 Conn_01x02, J8 Micro_SD_Card_Det1, J9 USB_C_Receptacle, Q1 NPN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

Commit message: raw placement
Parts:
- removed BZ1: Buzzer, Buzzer_Beeper:Buzzer_12x9.5RM7.6, symbol Device:Buzzer
- removed J13: Conn_01x02_Pin, Connector_PinHeader_2.00mm:PinHeader_1x02_P2.00mm_Vertical, symbol Connector:Conn_01x02_Pin
- removed J9: USB_C_Receptacle, IVS_FOOTPRINTS:USB_C_Receptacle_XKB_U262-16XN-4BVC11, symbol IVS_SYMBOLS:USB_C_Receptacle
- removed Q9: N_Mosfet, IVS_FOOTPRINTS:SOT23-3, symbol IVS_SYMBOLS:N_Mosfet
- removed R27: 1M, IVS_FOOTPRINTS:R_0603, symbol Device:R
Connections:
- no-connect marks 16 -> 12
Other:
- note removed: "BUZZER"
- note removed: "USB TYPE-C"
