File: PCB/74HC595_HEADER_OUTPUT.kicad_sch (KiCad schematic)
At the start: 38 parts, among them J1 Conn_01x03, J4 Conn_01x04, Q1 NPN, Q2 NPN, Q3 NPN, U2 74HC595

Commit message: layout pcb p2
Connections:
- net e: now reaches LE1.1 (e), LE2.1 (e), R8.2
- net f: now reaches LE1.10 (f), LE2.10 (f), R9.2
- net a: now reaches LE1.11 (a), LE2.11 (a), R4.2
- net d: now reaches LE1.2 (d), LE2.2 (d), R7.2
- net dot: now reaches LE1.3 (DPX), LE2.3 (DPX), R11.2
- net c: now reaches LE1.4 (c), LE2.4 (c), R6.2
- net g: now reaches LE1.5 (g), LE2.5 (g), R10.2
- net b: now reaches LE1.7 (b), LE2.7 (b), R5.2
Changed lines of the file:
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@@
     (company "NGUYỄN TRUNG THẢO")
   )
+  (bus_alias "SPI" (members "SCK" "MOSI" "MISO"))
   (bus_alias "I2C" (members "SDA" "SCL"))
-  (bus_alias "SPI" (members "SCK" "MOSI" "MISO"))
   (bus_alias "pLORA" (members "INT" "CS" "RST"))
   (junction (at 45.72 186.69) (diameter 0) (color 0 0 0 0)
@@
     (effects (font (size 1.27 1.27)) (justify left bottom))
   )
+  (label "f" (at 127.635 132.715 0) (fields_autoplaced)
+    (effects (font (size 1.27 1.27)) (justify left bottom))
+  )
   (label "LE7" (at 97.155 189.23 180) (fields_autoplaced)
     (effects (font (size 1.27 1.27)) (justify right bottom))
@@
     (effects (font (size 1.27 1.27)) (justify left bottom))
   )
+  (label "d" (at 127.635 127.635 0) (fields_autoplaced)
+    (effects (font (size 1.27 1.27)) (justify left bottom))
+  )
   (label "LE4" (at 160.02 231.14 0) (fields_autoplaced)
     (effects (font (size 1.27 1.27)) (justify left bottom))
@@
     (effects (font (size 1.27 1.27)) (justify left bottom))
   )
+  (label "dot" (at 127.635 137.795 0) (fields_autoplaced)
+    (effects (font (size 1.27 1.27)) (justify left bottom))
+  )
+  (label "e" (at 127.635 130.175 0) (fields_autoplaced)
+    (effects (font (size 1.27 1.27)) (justify left bottom))
+  )
+  (label "c" (at 127.635 125.095 0) (fields_autoplaced)
+    (effects (font (size 1.27 1.27)) (justify left bottom))
+  )
+  (label "g" (at 127.635 135.255 0) (fields_autoplaced)
+    (effects (font (size 1.27 1.27)) (justify left bottom))
+  )
   (label "LE1" (at 163.195 167.64 0) (fields_autoplaced)
     (effects (font (size 1.27 1.27)) (justify left bottom))
@@
     (effects (font (size 1.27 1.27)) (justify right bottom))
   )
+  (label "a" (at 127.635 120.015 0) (fields_autoplaced)
+    (effects (font (size 1.27 1.27)) (justify left bottom))
+  )
   (label "LE3" (at 97.155 199.39 180) (fields_autoplaced)
     (effects (font (size 1.27 1.27)) (justify right bottom))
   )
+  (label "b" (at 127.635 122.555 0) (fields_autoplaced)
+    (effects (font (size 1.27 1.27)) (justify left bottom))
+  )
   (hierarchical_label "LOG_TX" (shape output) (at 92.075 50.165 0) (fields_autoplaced)
