File: PCB/POWER.kicad_sch (KiCad schematic)
At the start: 24 parts, among them J2 Jack-DC, J3 Conn_01x07, Q10 P_Mosfet, U1 AMS1117, U1 XL1509

Commit message: raw placement
Parts:
- removed F2: Fuse, IVS_FOOTPRINTS:Fuse_1812_4532Metric, symbol IVS_SYMBOLS:Fuse
- removed J3: Conn_01x07, IVS_FOOTPRINTS:Conn_XH-P2.54mm-7P, symbol Connector_Generic:Conn_01x07
- C2: footprint IVS_FOOTPRINTS:C_0603_1608Metric -> IVS_FOOTPRINTS:C_0603
- C27: footprint IVS_FOOTPRINTS:C_0805 -> IVS_FOOTPRINTS:CP_EIA-3528-15_AVX-H
- Z1: footprint (none) -> IVS_FOOTPRINTS:D_MiniMELF
Connections:
- net GND: now also C2.2; no longer C2.1
- net VDC: now also C2.1; no longer C2.2
- no-connect marks 3 -> 0
Other:
- note added: "LDO 5V->3.3V"
- note added: "POWER INPUT AND IRREVESEABLE"
- note added: "SWITCHING BUCK CONVERTER 12V->5V"
- note removed: "POWER"
- moved on the sheet: C2, C24

Commit message: Update PCB
Connections:
- net A renamed VIN
Changed lines of the file:
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@@
   (junction (at 113.665 69.85) (diameter 0) (color 0 0 0 0)
   )
-  (junction (at 215.9 46.99) (diameter 0) (color 0 0 0 0)
-  )
   (junction (at 133.35 128.27) (diameter 0) (color 0 0 0 0)
   )
@@
   (junction (at 130.175 59.69) (diameter 0) (color 0 0 0 0)
   )
+  (junction (at 221.615 59.69) (diameter 0) (color 0 0 0 0)
+  )
   (junction (at 95.885 59.69) (diameter 0) (color 0 0 0 0)
   )
@@
     (stroke (width 0) (type default))
   )
-  (wire (pts (xy 215.9 46.99) (xy 215.9 59.69))
+  (wire (pts (xy 221.615 46.99) (xy 221.615 59.69))
     (stroke (width 0) (type default))
   )
@@
     (stroke (width 0) (type default))
   )
+  (wire (pts (xy 224.79 59.69) (xy 221.615 59.69))
+    (stroke (width 0) (type default))
+  )
   (wire (pts (xy 121.92 123.825) (xy 121.92 128.27))
     (stroke (width 0) (type default))
@@
     (stroke (width 0) (type default))
   )
+  (wire (pts (xy 221.615 59.69) (xy 215.9 59.69))
+    (stroke (width 0) (type default))
+  )
   (wire (pts (xy 127 128.27) (xy 127 128.905))
     (stroke (width 0) (type default))
@@
     (stroke (width 0) (type default))
   )
-  (wire (pts (xy 215.9 44.45) (xy 215.9 46.99))
+  (wire (pts (xy 224.79 56.515) (xy 224.79 59.69))
     (stroke (width 0) (type default))
   )
@@
     (stroke (width 0) (type default))
   )
-  (wire (pts (xy 165.1 46.99) (xy 215.9 46.99))
+  (wire (pts (xy 165.1 46.99) (xy 221.615 46.99))
     (stroke (width 0) (type default))
   )
@@
     (effects (font (size 3 3) (thickness 0.6) bold) (justify left bottom))
   )
-  (label "A" (at 85.09 59.69 0) (fields_autoplaced)
+  (label "VIN" (at 85.09 59.69 0) (fields_autoplaced)
     (effects (font (size 1.27 1.27)) (justify left bottom))
   )
@@
     )
   )
-  (symbol (lib_id "power:+5V") (at 215.9 44.45 0) (unit 1)
+  (symbol (lib_id "power:+5V") (at 224.79 56.515 0) (unit 1)
     (in_bom yes) (on_board yes) (dnp no) (fields_autoplaced)
-    (property "Reference" "#PWR05" (at 215.9 48.26 0)
-      (effects (font (size 1.27 1.27)) hide)
-    )
-    (property "Value" "+5V" (at 215.9 39.37 0)
+    (property "Reference" "#PWR05" (at 224.79 60.325 0)
+      (effects (font (size 1.27 1.27)) hide)
+    )
+    (property "Value" "+5V" (at 224.79 51.435 0)
       (effects (font (size 1.27 1.27)))
     )
-    (property "Footprint" "" (at 215.9 44.45 0)
-      (effects (font (size 1.27 1.27)) hide)
-    )
-    (property "Datasheet" "" (at 215.9 44.45 0)
-      (effects (font (size 1.27 1.27)) hide)
-    )
+    (property "Footprint" "" (at 224.79 56.515 0)
+      (effects (font (size 1.27 1.27)) hide)
+    )
+    (property "Datasheet" "" (at 224.79 56.515 0)
+      (effects (font (size 1.27 1.27)) hide)
+    )
