File: PCB/DO_AN_DKTD.kicad_pcb (KiCad board)
At the start: 2 copper layers, 96 x 97.2 mm, 164 parts, among them IC1 RTC_DS3231M, J1 Conn_01x07, J10 Jack-DC, J11 Conn_01x03_Pin, J12 Conn_01x03_Pin, J13 Conn_01x02_Pin, J2 Conn_01x02, J3 Conn_01x04, J4 Conn_01x03, J5 Conn_01x02, J6 , J7 Conn_01x05_Male, J8 Micro_SD_Card_Det1, J9 USB_C_Receptacle, Q1 NPN, Q10 P_Mosfet, Q2 NPN, Q3 NPN, Q4 NPN, Q5 NPN, Q6 NPN, Q7 NPN, Q8 NPN, Q9 N_Mosfet, SW1 RotaryEncoder_Switch, SW2 SW_Push, SW3 SW_Push, SW4 SW_Push, U1 AMS1117, U10 ESP-07, U2 74HC595, U3 PC817, U4 MOC3020M, U5 XL1509, U6 74HC595, U7 STM32F103C8Tx, U8 24C32N, U9 Ai-Thinker-Ra-02, Y1 Crystal_GND24_Small

Commit message: raw placement
Parts:
- removed C6: 10nF, IVS_FOOTPRINTS:C_0603
- removed D7: D_Schottky, IVS_FOOTPRINTS:D_SOD323
- removed F2: Fuse, IVS_FOOTPRINTS:Fuse_1812_4532Metric
- removed G*** (x2): LOGO, IVS_FOOTPRINTS:LoGo_ST_2.5x1.5mm
- removed G*** (x2): LOGO, IVS_FOOTPRINTS:LoGo_IDF_2.5x2.5mm
- removed G*** (x2): LOGO, IVS_FOOTPRINTS:LoGo_1412_10x8mm
- removed J1: Conn_01x07, IVS_FOOTPRINTS:Conn_XH-P2.54mm-7P
- removed J13: Conn_01x02_Pin, Connector_PinHeader_2.00mm:PinHeader_1x02_P2.00mm_Vertical
- removed J8: Micro_SD_Card_Det1, IVS_FOOTPRINTS:MicroSD_Socket_9P
- removed R19: 39, IVS_FOOTPRINTS:R_0603
- removed R55: 4k7, IVS_FOOTPRINTS:R_0603
- removed R60: 1M, IVS_FOOTPRINTS:R_0603
- removed REF** (x4): MountingHole_3.2mm_M3_Pad_Via, MountingHole:MountingHole_3.2mm_M3_Pad_Via
- removed REF**: ESD-Logo_6.6x6mm_SilkScreen, Symbol:ESD-Logo_6.6x6mm_SilkScreen
- removed U1: AMS1117, IVS_FOOTPRINTS:SOT233
- added R49: 1M, IVS_FOOTPRINTS:R_0603, F.Cu at (174.3, 131.3)
- added R52: 4k7, IVS_FOOTPRINTS:R_0603, F.Cu at (165.5, 120.5)
- added Ue: AMS1117, IVS_FOOTPRINTS:SOT233, F.Cu at (159.2, 51.2)
- added Z1: D_Zener, IVS_FOOTPRINTS:D_MiniMELF, F.Cu at (122.9, 50.1)
- BZ1: footprint Buzzer_Beeper:Buzzer_12x9.5RM7.6 -> IVS_FOOTPRINTS:Buzzer_12x9.5RM7.6
- C27: footprint IVS_FOOTPRINTS:C_0805 -> IVS_FOOTPRINTS:CP_EIA-3528-15_AVX-H
- D1: footprint IVS_FOOTPRINTS:Bridge_MB10F-13 -> IVS_FOOTPRINTS:DiodeBridge_MB10F-13AQ
- J11: footprint Connector_PinHeader_2.00mm:PinHeader_1x03_P2.00mm_Vertical -> IVS_FOOTPRINTS:PinHeader_1x03_P2.00mm_Vertical
- J12: value Conn_01x03_Pin -> Micro_SD_Card_Det1; footprint Connector_PinHeader_2.00mm:PinHeader_1x03_P2.00mm_Vertical -> IVS_FOOTPRINTS:MicroSD_Socket_9P
- J6: footprint Connector_PinHeader_2.54mm:PinHeader_1x06_P2.54mm_Vertical -> IVS_FOOTPRINTS:PinHeader_1x06_P2.54mm_Vertical
- J7: footprint Connector_PinHeader_2.54mm:PinHeader_1x05_P2.54mm_Vertical -> IVS_FOOTPRINTS:PinHeader_1x05_P2.54mm_Vertical
- R20: value 470 -> 22k
- R21: value 22k -> 470
- moved D2 111.0 mm to (99.1, 136.2), turned to 0 degrees
- moved J5 104.0 mm to (102.3, 126.4), turned to -90 degrees
- moved J2 102.9 mm to (102.3, 114.4), turned to -90 degrees
- moved R23 96.6 mm to (123.3, 139.8)
- moved F1 95.7 mm to (112.6, 134.9), turned to 90 degrees
- moved Q4 92.3 mm to (114.5, 141.7), turned to 0 degrees
- moved SW2 91.9 mm to (179.6, 50.7)
- moved D3 90.9 mm to (118.7, 140.9), turned to 0 degrees
- moved C23 87.2 mm to (187.3, 87.5), turned to 0 degrees
- moved C8 85.2 mm to (110.9, 117.5)
- moved R25 85.1 mm to (110.1, 128.3), turned to 0 degrees
- moved C22 85.1 mm to (187.3, 89.1), turned to 0 degrees
- moved SW3 85.0 mm to (175.5, 50.7), turned to -90 degrees
- moved U9 84.9 mm to (183.5, 99.6), turned to -90 degrees
- moved R20 83.8 mm to (110.1, 117.7)
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Connections:
- net /Peripheral/24C32.SCL renamed /74HC595_HEADER_OUTPUT/SHT31.SCL
- net /Peripheral/24C32.SDA renamed /74HC595_HEADER_OUTPUT/SHT31.SDA
- net /Peripheral/74HC595.OE renamed /74HC595_HEADER_OUTPUT/74HC595.OE
- net /Peripheral/74HC595.RCLK renamed /74HC595_HEADER_OUTPUT/74HC595.RCLK
- net /Peripheral/74HC595.SER renamed /74HC595_HEADER_OUTPUT/74HC595.SER
- net /Peripheral/74HC595.SRCLK renamed /74HC595_HEADER_OUTPUT/74HC595.SRCLK
- net /Peripheral/AC_DET renamed /STM32/ACDET
- net /Peripheral/Buzzer renamed /BUZZER/Buzzer
- net /Peripheral/Encoder.EnC_A renamed /STM32/ST.EnC_A
- net /Peripheral/Encoder.EnC_B renamed /STM32/ST.EnC_B
- net /Peripheral/Encoder.EnC_BT renamed /STM32/ST.EnC_BT
- net /Peripheral/L renamed /TRIAC_ACDET/L
- net /Peripheral/LE1 renamed /74HC595_HEADER_OUTPUT/LE1
- net /Peripheral/LE2 renamed /74HC595_HEADER_OUTPUT/LE2
- net /Peripheral/LE3 renamed /74HC595_HEADER_OUTPUT/LE3
- net /Peripheral/LE4 renamed /74HC595_HEADER_OUTPUT/LE4
- net /Peripheral/LE5 renamed /74HC595_HEADER_OUTPUT/LE5
- net /Peripheral/LE6 renamed /74HC595_HEADER_OUTPUT/LE6
- net /Peripheral/LE7 renamed /74HC595_HEADER_OUTPUT/LE7
- net /Peripheral/LOG_RX renamed /74HC595_HEADER_OUTPUT/LOG_RX
- net /Peripheral/LOG_TX renamed /74HC595_HEADER_OUTPUT/LOG_TX
- net /Peripheral/Load renamed /TRIAC_ACDET/Load
- net /Peripheral/N renamed /TRIAC_ACDET/N
- net /Peripheral/TRIAC renamed /STM32/TRIAC
- net /Peripheral/TYPE_C.D+ renamed /STM32/ST.D+
- net /Peripheral/TYPE_C.D- renamed /STM32/ST.D-
- net /Peripheral/Vbat renamed /RTC_DS3231/Vbat
- C25 pad 1: GND -> VDC
- C25 pad 2: VDC -> GND
- D2 pad 2: /Peripheral/L_after -> /TRIAC_ACDET/L_after
- D5 pad 1: /Peripheral/SD.DET -> /MICRO_SD/SD.DET
- D5 pad 3: /Peripheral/SD.CS -> /MICRO_SD/SD.CS
- D5 pad 4: /Peripheral/LORA.MOSI -> /LORA/LORA.MOSI
- D5 pad 5: /Peripheral/LORA.SCK -> /LORA/LORA.SCK
- D5 pad 6: /Peripheral/LORA.MISO -> /LORA/LORA.MISO
- F1 pad 1: /Peripheral/L_after -> /TRIAC_ACDET/L_after
- J12 pad 1: /Peripheral/LORA.MISO -> unconnected-(J12-DAT2-Pad1)
- J12 pad 2: /Peripheral/LORA.SCK -> /MICRO_SD/SD.CS
- J12 pad 3: /Peripheral/LORA.MOSI -> /LORA/LORA.MOSI
- R20 pad 1: Net-(C8-Pad1) -> Net-(D1-+)
- R20 pad 2: /Peripheral/L_after -> Net-(D1--)
- R21 pad 1: Net-(D1-+) -> Net-(C8-Pad1)
- R21 pad 2: Net-(D1--) -> /TRIAC_ACDET/L_after
- R6 pad 2: /Peripheral/L_after -> /TRIAC_ACDET/L_after
- U7 pad 27: /Peripheral/SD.CS -> /MICRO_SD/SD.CS
- U7 pad 28: /Peripheral/SD.DET -> /MICRO_SD/SD.DET
- U7 pad 38: /Peripheral/LORA.CS -> /STM32/LORA.CS
- U7 pad 39: /Peripheral/LORA.SCK -> /STM32/ST.SCK
- U7 pad 40: /Peripheral/LORA.MISO -> /STM32/ST.MISO
- U7 pad 41: /Peripheral/LORA.MOSI -> /STM32/ST.MOSI
- U7 pad 42: /Peripheral/LORA.INT -> /STM32/LORA.INT
- U7 pad 43: /Peripheral/LORA.RST -> /STM32/LORA.RST
- U9 pad 12: /Peripheral/LORA.SCK -> /LORA/LORA.SCK
- U9 pad 13: /Peripheral/LORA.MISO -> /LORA/LORA.MISO
- U9 pad 14: /Peripheral/LORA.MOSI -> /LORA/LORA.MOSI
- U9 pad 15: /Peripheral/LORA.CS -> /LORA/LORA.CS
- U9 pad 4: /Peripheral/LORA.RST -> /LORA/LORA.RST
- U9 pad 5: /Peripheral/LORA.INT -> /LORA/LORA.INT
Routing:
- net +3V3: track 368.7 -> 0.00 mm, vias 22 -> 0
- net +5V: track 172.7 -> 0.00 mm, vias 8 -> 0
- net /Peripheral/LORA.MOSI: track 76.7 -> 0.00 mm, vias 2 -> 0
- net /STM32/TRIAC: track 75.5 -> 0.00 mm
- net /74HC595_HEADER_OUTPUT/SHT31.SCL: track 72.8 -> 0.00 mm, vias 3 -> 0
- net /74HC595_HEADER_OUTPUT/SHT31.SDA: track 71.8 -> 0.00 mm, vias 3 -> 0
- net /Peripheral/LORA.SCK: track 67.4 -> 0.00 mm, vias 2 -> 0
- net /ESP/TX_ESP32: track 67.0 -> 0.00 mm
- net /STM32/RST: track 64.5 -> 0.00 mm, vias 2 -> 0
- net /STM32/ST.EnC_BT: track 63.6 -> 0.00 mm, vias 2 -> 0
- net /STM32/ACDET: track 61.4 -> 0.00 mm
- net /Peripheral/LORA.MISO: track 60.0 -> 0.00 mm, vias 2 -> 0
- net /Peripheral/SD.CS: track 59.5 -> 0.00 mm, vias 2 -> 0
- net /STM32/ST.EnC_A: track 56.4 -> 0.00 mm, vias 1 -> 0
- net Net-(LE1-a): track 53.9 -> 0.00 mm
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- removed copper zone on F.Cu, net +3V3
- removed copper zone on F.Cu, net +5V
- removed copper zone on F.Cu, net /POWER/5vin
- removed copper zone on F.Cu, net /POWER/A
- removed copper zone on F.Cu, net /POWER/B
- removed copper zone on F.Cu, net /POWER/VOUT
- removed copper zone on B.Cu, net GND
- removed copper zone on F.Cu, net GND
- removed copper zone on F.Cu, net VDC
Other:
- outline, holes or cut-outs redrawn
- board text removed: "1"
- board text removed: "12V IN"
- board text removed: "2"
- board text removed: "3"
- board text removed: "3V B RX TX R G"
- board text removed: "3V SCL SDA G"
- board text removed: "3V3"
- board text removed: "5V"
- board text removed: "5V 3V G IO CLK"
- board text removed: "BOOT"
- board text removed: "BORAD V0.1 Designed By Nguyen Trung Thao 20151564"
- board text removed: "D+"
- board text removed: "D-"
- board text removed: "G RX TX"
- board text removed: "I2C"
- board text removed: "IN"
- board text removed: "MI"
- board text removed: "MO"
- board text removed: "OUT"
- board text removed: "RST"
- board text removed: "SCK"
- board text removed: "UART"
- board text removed: "USB"
- board text removed: "~220V"

Commit message: layout pcb p2
Parts:
- moved R14 6.30 mm to (171.5, 99.5)
- moved R17 6.30 mm to (171.5, 107.4)
- moved R13 6.30 mm to (171.5, 96.8)
- moved R15 6.30 mm to (171.5, 102.1)
- moved R16 6.30 mm to (171.5, 104.8)
- moved C29 0.50 mm to (174.8, 73.3)
Changed lines of the file:
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@@
   )
   (footprint "IVS_FOOTPRINTS:R_0603" (layer "F.Cu")
-    (at 169.925 98.65)
+    (at 171.5 104.75)
     (property "Field2" "")
     (property "Sheetfile" "74HC595_HEADER_OUTPUT.kicad_sch")
@@
   )
   (footprint "IVS_FOOTPRINTS:R_0603" (layer "F.Cu")
-    (at 169.925 93.35)
+    (at 171.5 99.45)
     (property "Field2" "")
     (property "Sheetfile" "74HC595_HEADER_OUTPUT.kicad_sch")
@@
   )
   (footprint "IVS_FOOTPRINTS:R_0603" (layer "F.Cu")
-    (at 169.925 96)
+    (at 171.5 102.1)
     (property "Field2" "")
     (property "Sheetfile" "74HC595_HEADER_OUTPUT.kicad_sch")
@@
         (effects (font (size 1 1) (thickness 0.15)))
     )
-    (fp_text user "${REFERENCE}" (at 0 0.1 90) (layer "F.Fab") hide
-        (effects (font (size 0.6 0.6) (thickness 0.09)))
-    )
     (fp_text user "${REFERENCE}" (at 0 2.5 90 unlocked) (layer "F.Fab") hide
         (effects (font (size 1 1) (thickness 0.15)))
     )
+    (fp_text user "${REFERENCE}" (at 0 0.1 90) (layer "F.Fab") hide
+        (effects (font (size 0.6 0.6) (thickness 0.09)))
+    )
     (fp_line (start -2.1625 -1.775) (end -2.1625 -1.655)
       (stroke (width 0.25) (type solid)) (layer "F.SilkS"))
@@
   )
   (footprint "IVS_FOOTPRINTS:R_0603" (layer "F.Cu")
-    (at 169.925 101.3)
+    (at 171.5 107.4)
     (property "Field2" "")
     (property "Sheetfile" "74HC595_HEADER_OUTPUT.kicad_sch")
@@
       (stroke (width 0.01) (type solid)) (fill solid) (layer "F.Fab"))
     (dimension (type aligned) (layer "Dwgs.User")
-      (pts (xy 127.4 114.315) (xy 127.4 118.2266))
-      (height 4.87)
-      (gr_text "0.1540 in" (at 121.38 116.2708 90) (layer "Dwgs.User")
+      (pts (xy 136.925 113.4708) (xy 136.925 119.0708))
+      (height -3.705)
+      (gr_text "0.2205 in" (at 139.48 116.2708 90) (layer "Dwgs.User")
         (effects (font (size 1 1) (thickness 0.15)))
       )
@@
     )
     (dimension (type aligned) (layer "Dwgs.User")
-      (pts (xy 136.925 113.4708) (xy 136.925 119.0708))
-      (height -3.705)
-      (gr_text "0.2205 in" (at 139.48 116.2708 90) (layer "Dwgs.User")
+      (pts (xy 127.4 114.315) (xy 127.4 118.2266))
+      (height 4.87)
+      (gr_text "0.1540 in" (at 121.38 116.2708 90) (layer "Dwgs.User")
         (effects (font (size 1 1) (thickness 0.15)))
       )
@@
   )
   (footprint "IVS_FOOTPRINTS:R_0603" (layer "F.Cu")
-    (at 169.925 90.7)
+    (at 171.5 96.8)
     (property "Field2" "")
     (property "Sheetfile" "74HC595_HEADER_OUTPUT.kicad_sch")
@@
         (effects (font (size 1 1) (thickness 0.15)))
     )
-    (fp_text user "${REFERENCE}" (at 0 0.1) (layer "F.Fab") hide
-        (effects (font (size 0.6 0.6) (thickness 0.09)))
-    )
     (fp_text user "${REFERENCE}" (at 0 2.5 180 unlocked) (layer "F.Fab") hide
         (effects (font (size 1 1) (thickness 0.15)))
     )
+    (fp_text user "${REFERENCE}" (at 0 0.1) (layer "F.Fab") hide
+        (effects (font (size 0.6 0.6) (thickness 0.09)))
+    )
     (fp_line (start -2.1625 -1.775) (end -2.1625 -1.655)
       (stroke (width 0.25) (type solid)) (layer "F.SilkS"))
@@
       (stroke (width 0.01) (type solid)) (fill solid) (layer "F.Fab"))
     (dimension (type aligned) (layer "Dwgs.User")
-      (pts (xy 127.395 107.4866) (xy 137.555 107.4866))
-      (height 4.7442)
-      (gr_text "0.4000 in" (at 132.475 111.0808) (layer "Dwgs.User")
+      (pts (xy 136.92 102.7308) (xy 136.92 108.3308))
+      (height -3.705)
+      (gr_text "0.2205 in" (at 139.475 105.5308 90) (layer "Dwgs.User")
         (effects (font (size 1 1) (thickness 0.15)))
       )
@@
     )
     (dimension (type aligned) (layer "Dwgs.User")
-      (pts (xy 127.395 103.575) (xy 127.395 107.4866))
-      (height 4.87)
-      (gr_text "0.1540 in" (at 121.375 105.5308 90) (layer "Dwgs.User")
+      (pts (xy 127.395 107.4866) (xy 137.555 107.4866))
+      (height 4.7442)
+      (gr_text "0.4000 in" (at 132.475 111.0808) (layer "Dwgs.User")
         (effects (font (size 1 1) (thickness 0.15)))
       )
@@
     )
     (dimension (type aligned) (layer "Dwgs.User")
-      (pts (xy 136.92 102.7308) (xy 136.92 108.3308))
-      (height -3.705)
-      (gr_text "0.2205 in" (at 139.475 105.5308 90) (layer "Dwgs.User")
+      (pts (xy 127.395 103.575) (xy 127.395 107.4866))
+      (height 4.87)
+      (gr_text "0.1540 in" (at 121.375 105.5308 90) (layer "Dwgs.User")
         (effects (font (size 1 1) (thickness 0.15)))
       )
@@
         (effects (font (size 1 1) (thickness 0.15)))
     )
-    (fp_text user "${REFERENCE}" (at 0 2.5 -90 unlocked) (layer "F.Fab") hide
-        (effects (font (size 1 1) (thickness 0.15)))
-    )
     (fp_text user "${REFERENCE}" (at 0 0.1 90) (layer "F.Fab") hide
         (effects (font (size 0.6 0.6) (thickness 0.09)))
     )
+    (fp_text user "${REFERENCE}" (at 0 2.5 -90 unlocked) (layer "F.Fab") hide
+        (effects (font (size 1 1) (thickness 0.15)))
+    )
     (fp_line (start -2.1625 -1.775) (end -2.1625 -1.655)
       (stroke (width 0.25) (type solid)) (layer "F.SilkS"))
@@
     (pad "4" smd roundrect (at -1.1 -0.85 225) (size 1.4 1.2) (layers "F.Cu" "F.Paste" "F.Mask") (roundrect_rratio 0.05)
       (net 2 "GND") (pinfunction "4") (pintype "passive"))
-    (model "${IOTVISION_3D}/Crystal/SMD/Crystal_SMD_3225/3225 SMD Crystal Oscillator.STEP"
+    (model "${IOTVISION_3D}/Crystal/SMD/Crystal_SMD_5032-4Pin_5.0x3.2mm/Crystal_SMD_5032-4Pin_5.0x3.2mm.wrl"
       (offset (xyz 0 0 0))
       (scale (xyz 1 1 1))
-      (rotate (xyz -90 0 0))
+      (rotate (xyz 0 0 0))
     )
   )
@@
   )
   (footprint "IVS_FOOTPRINTS:C_0603" (layer "F.Cu")
-    (at 174.8 72.8 180)
+    (at 174.8 73.3 180)
     (property "Sheetfile" "ESP.kicad_sch")
     (property "Sheetname" "ESP")
@@
         (effects (font (size 1 1) (thickness 0.15)))
     )
-    (fp_text user "KEEP-OUT ZONE" (at 8.15 -5.05 90) (layer "Cmts.User")
+    (fp_text user "Antenna" (at 8.06 -2.5 90) (layer "Cmts.User")
         (effects (font (size 1 1) (thickness 0.15)))
     )
-    (fp_text user "Antenna" (at 8.06 -2.5 90) (layer "Cmts.User")
+    (fp_text user "KEEP-OUT ZONE" (at 8.15 -5.05 90) (layer "Cmts.User")
         (effects (font (size 1 1) (thickness 0.15)))
     )
@@
     (style (thickness 0.1) (arrow_length 1.27) (text_position_mode 0) (extension_height 0.58642) (extension_offset 0.5) keep_text_aligned)
   )
-  (group "" (id 56304402-bffe-417f-ac64-b0ace4b4ea6a)
-    (members
-      0f735d15-511b-45a0-8482-8a0aea9a1c58
-      26a82977-800a-4232-947e-958b1692b029
-      2ff1b721-b9d8-4f00-9f50-e4a74940130f
-      5dd663e9-de11-4ae2-bb21-092370cce3b8
-      6980b9fa-51cf-43b4-9abd-1483c5fe94b9
-      88483a23-1ec9-4d6d-979d-ece309d7d630
-      a5a195ed-a6bf-4c31-8e83-ef4e25219efb
-      d87fe76b-4b35-4027-a5a3-69c98441c7f5
-      ec996437-19bd-40e3-b05f-02872efa9670
-    )
-  )
-  (group "" (id ccd8118d-26f2-46a5-96f8-40bd7d74eaa9)
-    (members
-      333c6035-5e0d-4342-96ee-e41d6dbad678
-      4feb773b-3fc0-4d6f-b012-ed4ea3d5c2ac
-      9a3aa83f-d9e8-4475-9746-3b9d9c6141ac
-    )
-  )
-  (group "" (id ec15af60-665b-4c3d-bab9-04b3f1b5ed74)
-    (members
-      1681b70b-55fe-472a-8149-1f17cc50a896
-      2bf675c9-991a-4afb-bc37-c724e001b778
-      6bc88161-b957-451e-9112-8587fe0a5e55
-    )
-  )
 )

Commit message: Update PCB
Parts:
- removed Ue: AMS1117, IVS_FOOTPRINTS:SOT233
- added U1: AMS1117, IVS_FOOTPRINTS:SOT233, F.Cu at (158.8, 51.5)
- moved R15 48.0 mm to (124.1, 109.4)
- moved R17 47.7 mm to (124.1, 102.0)
- moved R13 47.5 mm to (124.1, 100.2)
- moved R14 47.4 mm to (124.1, 98.4)
- moved R16 47.4 mm to (124.1, 105.7)
- moved R25 37.7 mm to (146.2, 139.2), turned to 180 degrees
- moved R24 36.2 mm to (146.3, 125.7), turned to -90 degrees
- moved R47 32.0 mm to (131.0, 66.4), turned to -90 degrees
- moved Q6 31.0 mm to (130.7, 94.2), turned to -90 degrees
- moved Q1 30.7 mm to (130.7, 108.2), turned to -90 degrees
- moved R48 30.7 mm to (133.0, 66.4), turned to -90 degrees
- moved U6 30.0 mm to (113.5, 92.8)
- moved R44 29.6 mm to (135.0, 66.4), turned to -90 degrees
- moved LE4 28.0 mm to (131.0, 69.9), turned to 90 degrees
- moved Q8 27.2 mm to (130.7, 86.7), turned to -90 degrees
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Connections:
- net /POWER/A renamed /POWER/VIN
- net Net-(LE1-DPX) renamed /74HC595_HEADER_OUTPUT/dot
- net Net-(LE1-a) renamed /74HC595_HEADER_OUTPUT/a
- net Net-(LE1-b) renamed /74HC595_HEADER_OUTPUT/b
- net Net-(LE1-c) renamed /74HC595_HEADER_OUTPUT/c
- net Net-(LE1-d) renamed /74HC595_HEADER_OUTPUT/d
- net Net-(LE1-e) renamed /74HC595_HEADER_OUTPUT/e
- net Net-(LE1-f) renamed /74HC595_HEADER_OUTPUT/f
- net Net-(LE1-g) renamed /74HC595_HEADER_OUTPUT/g
- U7 pad 39: /STM32/ST.SCK -> /LORA/LORA.SCK
- U7 pad 40: /STM32/ST.MISO -> /LORA/LORA.MISO
- U7 pad 41: /STM32/ST.MOSI -> /LORA/LORA.MOSI
Routing:
- net +3V3: track 0.00 -> 367.2 mm, vias 0 -> 24
- net GND: track 0.00 -> 145.8 mm, vias 0 -> 82
- net +5V: track 0.00 -> 124.3 mm, vias 0 -> 11
- net /LORA/LORA.MISO: track 0.00 -> 121.4 mm
- net /LORA/LORA.SCK: track 0.00 -> 112.2 mm, vias 0 -> 2
- net /LORA/LORA.MOSI: track 0.00 -> 104.1 mm
- net /74HC595_HEADER_OUTPUT/SHT31.SCL: track 0.00 -> 102.9 mm, vias 0 -> 4
- net /74HC595_HEADER_OUTPUT/SHT31.SDA: track 0.00 -> 92.1 mm, vias 0 -> 2
- net /STM32/ST.EnC_BT: track 0.00 -> 90.9 mm, vias 0 -> 2
- net /74HC595_HEADER_OUTPUT/LOG_RX: track 0.00 -> 86.3 mm, vias 0 -> 2
- net /STM32/TRIAC: track 0.00 -> 80.6 mm, vias 0 -> 2
- net /BUZZER/Buzzer: track 0.00 -> 80.3 mm, vias 0 -> 2
- net /74HC595_HEADER_OUTPUT/LOG_TX: track 0.00 -> 78.8 mm, vias 0 -> 4
- net /MICRO_SD/SD.DET: track 0.00 -> 77.3 mm, vias 0 -> 4
- net /MICRO_SD/SD.CS: track 0.00 -> 76.0 mm, vias 0 -> 3
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- added copper zone on F.Cu, net +3V3
- added copper zone on F.Cu, net +5V
- added copper zone on F.Cu, net /POWER/B
- added copper zone on F.Cu, net /POWER/VIN
- added copper zone on F.Cu, net /POWER/VOUT
- added copper zone on B.Cu, net /TRIAC_ACDET/L_after
- added copper zone on F.Cu, net /TRIAC_ACDET/L_after
- added copper zone on B.Cu, net GND
- added copper zone on F.Cu, net GND
- added copper zone on F.Cu, net VDC
Other:
- outline, holes or cut-outs redrawn
- board text added: "12V+"
- board text added: "220~"
- board text added: "3V3"
- board text added: "BOOT RST"
- board text added: "GND"
- board text added: "LOAD"
- board text added: "RX"
- board text added: "SCL"
- board text added: "SDA"
- board text added: "TX"

Commit message: Mini layout p3
Parts:
- moved C9 3.10 mm to (107.0, 90.8), turned to 90 degrees
- moved C30 0.33 mm to (169.8, 76.3)
- moved R33 0.11 mm to (172.0, 76.2)
- moved R42 0.07 mm to (176.9, 76.2)
- moved R34 0.07 mm to (173.6, 76.2)
- moved R35 0.05 mm to (175.3, 76.2)
Routing:
- net +5V: track 124.3 -> 393.7 mm, vias 11 -> 18
- net +3V3: track 367.2 -> 482.0 mm, vias 24 -> 27
- net GND: track 145.8 -> 212.6 mm, vias 82 -> 101
- net /74HC595_HEADER_OUTPUT/g: track 51.7 -> 64.8 mm
- net /ESP/RST: track 40.9 -> 53.0 mm
- net /74HC595_HEADER_OUTPUT/c: track 47.9 -> 58.5 mm
- net /74HC595_HEADER_OUTPUT/dot: track 44.2 -> 52.7 mm
- net /74HC595_HEADER_OUTPUT/d: track 41.2 -> 46.4 mm
- net Net-(LE2-CC1): track 23.5 -> 26.0 mm
- net Net-(LE2-CC3): track 37.8 -> 39.0 mm
- net Net-(LE1-CC1): track 36.6 -> 37.6 mm
- net Net-(U7-PB11): track 12.0 -> 12.7 mm
- net Net-(IC1-VBAT): track 18.9 -> 19.5 mm
- net Net-(U10-GPIO2): track 11.9 -> 12.5 mm
- net Net-(LE1-CC2): track 45.5 -> 46.0 mm
- added copper zone on B.Cu, net +5V
