File: PCB/DO_AN_DKTD.kicad_sch (KiCad schematic)
At the start: 0 parts

Commit message: raw placement
Other:
- sheet Peripheral renamed 74HC595_HEADER_OUTPUT
- added sheet BUZZER (BUZZER.kicad_sch)
- added sheet EEPROM (EEPROM.kicad_sch)
- added sheet LORA (LORA.kicad_sch)
- added sheet MICRO_SD (MICRO_SD.kicad_sch)
- added sheet RTC_DS3231 (RTC_DS3231.kicad_sch)
- added sheet TRIAC_ACDET (TRIAC_ACDET.kicad_sch)
- added sheet TYPE C (TYPE C.kicad_sch)
- added sheet encoder (encoder.kicad_sch)
- sheet 74HC595_HEADER_OUTPUT: file Peripheral.kicad_sch -> 74HC595_HEADER_OUTPUT.kicad_sch
- sheet 74HC595_HEADER_OUTPUT ports: added none; removed 24C32{I2C}, AC_DET, Buzzer, DS3231{I2C}, Encoder{EnC}, LORA{SPI}, LORA{pLORA}, SD{SPI}, SD{pSD}, TRIAC, TYPE_C{USB}

Commit message: Update PCB
Changed lines of the file:
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@@
     (stroke (width 0) (type default))
   )
-  (bus (pts (xy 184.785 164.465) (xy 192.405 164.465))
+  (bus (pts (xy 184.785 158.75) (xy 192.405 158.75))
     (stroke (width 0) (type default))
   )
@@
     (stroke (width 0) (type default))
   )
-  (bus (pts (xy 192.405 164.465) (xy 192.405 55.245))
+  (bus (pts (xy 192.405 158.75) (xy 192.405 55.245))
     (stroke (width 0) (type default))
   )
