File: PCB/MICRO_SD.kicad_sch (KiCad schematic)
At the start: 4 parts, among them J8 Micro_SD_Card_Det1

Commit message: Update some footprints name
Parts:
- J8: footprint IVS_FOOTPRINTS:MicroSD_Socket_9P -> IVS_FOOTPRINTS:Socket_MicroSD-9P
Changed lines of the file:
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@@
       (effects (font (size 1.27 1.27)))
     )
-    (property "Footprint" "IVS_FOOTPRINTS:MicroSD_Socket_9P" (at 217.805 72.39 0)
+    (property "Footprint" "IVS_FOOTPRINTS:Socket_MicroSD-9P" (at 217.805 72.39 0)
       (effects (font (size 1.27 1.27)) hide)
     )
