File: PCB/STM32.kicad_sch (KiCad schematic)
At the start: 26 parts, among them J11 Conn_01x03_Pin, J3 Conn_01x05_Male, SW2 SW_Push, U4 STM32F103C8Tx, Y1 Crystal_GND24_Small

Commit message: raw placement
Parts:
- J11: footprint Connector_PinHeader_2.00mm:PinHeader_1x03_P2.00mm_Vertical -> IVS_FOOTPRINTS:PinHeader_1x03_P2.00mm_Vertical
- J3: footprint Connector_PinHeader_2.54mm:PinHeader_1x05_P2.54mm_Vertical -> IVS_FOOTPRINTS:PinHeader_1x05_P2.54mm_Vertical
Changed lines of the file:
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@@
       (effects (font (size 1.27 1.27)) hide)
     )
-    (property "Footprint" "Connector_PinHeader_2.00mm:PinHeader_1x03_P2.00mm_Vertical" (at 116.205 157.48 0)
+    (property "Footprint" "IVS_FOOTPRINTS:PinHeader_1x03_P2.00mm_Vertical" (at 116.205 157.48 0)
       (effects (font (size 1.27 1.27)) hide)
     )
@@
       (effects (font (size 1.27 1.27)) hide)
     )
-    (property "Footprint" "Connector_PinHeader_2.54mm:PinHeader_1x05_P2.54mm_Vertical" (at 278.13 76.835 0)
-      (effects (font (size 1.27 1.27)) hide)
-    )
+    (property "Footprint" "IVS_FOOTPRINTS:PinHeader_1x05_P2.54mm_Vertical" (at 278.13 76.835 0)
+      (effects (font (size 1.27 1.27)) hide)
+    )

Commit message: Update some footprints name
Parts:
- Y1: footprint IVS_FOOTPRINTS:Crystal_3225_4P_3.2x2.6mm -> IVS_FOOTPRINTS:Crystal-SMD-4P-3.2x2.6mm-3225
Changed lines of the file:
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@@
       (effects (font (size 1.27 1.27)) hide)
     )
-    (property "Footprint" "IVS_FOOTPRINTS:Crystal_3225_4P_3.2x2.6mm" (at 196.85 79.375 0)
+    (property "Footprint" "IVS_FOOTPRINTS:Crystal-SMD-4P-3.2x2.6mm-3225" (at 196.85 79.375 0)
       (effects (font (size 1.27 1.27)) hide)
     )
